File: m68030-bbb.kicad_sch (KiCad schematic)
At the start: 13 parts, among them U1 MC68030, U10 M29F160F, U11 M29F160F, U12 XC95108TQ100, U13 SST39SF010, U2 R68561, U3 68230, U4 CY62167GN-45ZXI, U5 CY62167GN-45ZXI, U6 CY62167GN-45ZXI, U7 CY62167GN-45ZXI, U8 M29F160F, U9 M29F160F

Commit message: Pretty much finished with the glue logic.  Doing intc now.
Parts:
- added TP1, TP11, TP2, TP7: TestPoint_Small, TestPoint:TestPoint_Loop_D2.50mm_Drill1.0mm, symbol Connector:TestPoint_Small
- added TP10, TP12, TP14, TP4, TP5, TP6, TP8, TP9: PGND, Rassilon:TestPoint_2Pads_Pitch2.54mm_Drill0.8mm_tie_bottom, symbol Connector:TestPoint_2Pole
- added TP13: OCS, TestPoint:TestPoint_Loop_D2.50mm_Drill1.0mm, symbol Connector:TestPoint_Small
- added TP3: PND, TestPoint:TestPoint_Loop_D2.50mm_Drill1.0mm, symbol Connector:TestPoint_Small
Connections:
- net SYSCLK is gone; now on net ~{AS}: U12.23 (FB1_M14_GCLK2)
- net +5V: now also U10.37 (VCC), U11.37 (VCC), U4.12 (CE2), U4.14 (UB#), U4.15 (LB#), U4.37 (VCC), U5.12 (CE2), U5.14 (UB#), U5.15 (LB#), U5.37 (VCC), U6.12 (CE2), U6.14 (UB#), U6.15 (LB#), U6.37 (VCC), U7.12 (CE2), U7.14 (UB#), U7.15 (LB#), U7.37 (VCC), U8.37 (VCC), U9.37 (VCC)
- net A0: now also U12.25 (FB1_M15), U3.29 (RS1)
- net A1: now also U12.28 (FB1_M17), U2.10 (A1), U3.28 (RS2)
- net A2: now also U10.45 (A-1/D15), U11.45 (A-1/D15), U2.13 (A2), U3.27 (RS3), U9.45 (A-1/D15)
- net A20: now also U12.65 (FB6_M2)
- net A21: now also U12.66 (FB6_M3)
- net A22: now also U12.67 (FB6_M5)
- net A23: now also U12.68 (FB6_M6)
- net A24: now also U12.70 (FB6_M8)
- net A25: now also U12.71 (FB6_M9)
- net A26: now also U12.72 (FB6_M11)
- net A27: now also U12.73 (FB6_M4)
- net A28: now also U12.74 (FB6_M12)
- net A29: now also U12.76 (FB6_M14)
- net A3: now also U2.14 (A3), U3.26 (RS4)
- net A30: now also U12.77 (FB6_M15)
- net A31: now also U12.78 (FB6_M17)
- net A4: now also U2.12 (A4), U3.25 (RS5)
- net D24: now also U3.44 (D0)
- net D25: now also U3.45 (D1)
- net D26: now also U3.46 (D2)
- net D27: now also U3.47 (D3)
- net D28: now also U3.48 (D4)
- net D29: now also U3.1 (D5)
- net D30: now also U3.2 (D6)
- net D31: now also U3.3 (D7)
- net GND: now also U10.47 (~{BYTE}), U11.47 (~{BYTE}), U3.38 (GND), U8.47 (~{BYTE}), U9.47 (~{BYTE}), TP10.2, TP12.2, TP14.2, TP4.2, TP5.2, TP6.2, TP8.2, TP9.2; no longer U13.24 (OE)
- net R/~{W}: now also U12.15 (FB1_M5), U2.22 (R/~{W}), U3.43 (R/W); no longer U12.17 (FB1_M8), U13.31 (PGM)
- net ~{AS}: no longer U12.15 (FB1_M5)
- net ~{CBACK}: now also U12.96 (FB2_M2)
- net ~{CBREQ}: now also U12.97 (FB2_M3)
- net ~{CIIN}: now also U12.16 (FB1_M6)
- net ~{CIOUT}: now also U12.17 (FB1_M8)
- net ~{DS}: now also U12.18 (FB1_M9); no longer U12.16 (FB1_M6)
- net ~{M230CE}: now also U3.41 (CS)
- net ~{R561CE}: now also U2.44 (~{CS})
- net ~{RDLL}: now also U12.33 (FB3_M6)
- net ~{RDLM}: now also U12.32 (FB3_M5)
- net ~{RDUM}: now also U12.30 (FB3_M3)
- net ~{RDUU}: now also U12.29 (FB3_M2)
- net ~{RESET}: now also U10.12 (~{RST}), U11.12 (~{RST}), U12.1 (FB2_M6), U2.31 (~{RESET}), U3.39 (RESET), U8.12 (~{RST}), U9.12 (~{RST})
- net ~{WELL}: now also U12.37 (FB3_M11)
- net ~{WELM}: now also U12.36 (FB3_M9)
- net ~{WEUM}: now also U12.35 (FB3_M8)
- net ~{WEUU}: now also U12.34 (FB3_M4)
- net ~{UDS}: now reaches U2.1 (~{UDS})
- net ~{UDS}: now also U12.39 (FB3_M12)
- net ~{R561DTACK}: now reaches U2.2 (~{DTACK})
- net ~{R561DTACK}: now also U12.95 (FB4_M17)
- net ~{LDS}: now reaches U2.47 (~{LDS})
- net ~{LDS}: now also U12.40 (FB3_M14)
- net ~{WR}: now reaches U12.11 (FB2_M16)
- net ~{WR}: now also U13.31 (PGM)
- net ~{RD}: now reaches U12.12 (FB2_M17)
- net ~{RD}: now also U13.24 (OE)
- net ~{IOSEL}: now reaches U12.2 (FB2_M4)
- net ~{IOSEL}: now also U12.4 (FB2_M9_GTS2)
- net at U12.3 (FB2_M8_GTS1): now also TP2.1
- net at U12.41 (FB3_M15): now also TP13.1
- net ~{IOCS0}: now reaches U12.42 (FB3_M16)
- net ~{IOCS1}: now reaches U12.49 (FB3_M17)
- net at U12.79 (FB6_M16): now also TP1.1
- net at U12.80 (FB4_M4): now also TP5.1
- net at U12.81 (FB4_M2): now also TP3.1
- net at U12.82 (FB4_M3): now also TP4.1
- net at U12.85 (FB4_M5): now also TP6.1
- net at U12.86 (FB4_M6): now also TP7.1
- net at U12.87 (FB4_M8): now also TP8.1
- net at U12.89 (FB4_M9): now also TP9.1
- net at U12.90 (FB4_M11): now also TP10.1
- net at U12.91 (FB4_M12): now also TP11.1
- net at U12.92 (FB4_M16): now also TP14.1
- net at U12.93 (FB4_M14): now also TP12.1
- net ~{M230DTACK}: now reaches U12.94 (FB4_M15)
- net ~{M230DTACK}: now also U3.42 (DTACK)
- net CLK8MHz: now reaches U3.40 (CLK)
- net SYSCLK2X renamed ~{CPUCLK}
- no-connect marks 1 -> 3
Other:
- moved on the sheet: U10, U11, U8, U9
